Commit message: optimal some functions and urdf file

File: data/fr3_capsule.urdf (robot description, URDF)
Before this commit: robot fr3, 11 links, 10 joints
Links:
- added link fr3_hand, mass 0.73; collision mesh filename=package://franka_description/meshes/robot_ee/franka_hand_wh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; visual mesh filename=package://franka_description/meshes/robot_ee/franka_hand_wh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
- added link fr3_link0, mass 2.3966; collision mesh filename=package://franka_description/meshes/robot_arms/fr3/collisio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; visual mesh filename=package://franka_description/meshes/robot_arms/fr3/visual/l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
- added link fr3_link1, mass 2.9274653454; collision mesh filename=package://franka_description/meshes/robot_arms/fr3/collisio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; visual mesh filename=package://franka_description/meshes/robot_arms/fr3/visual/l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
- added link fr3_link2, mass 2.9355370338; collision mesh filename=package://franka_description/meshes/robot_arms/fr3/collisio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; visual mesh filename=package://franka_description/meshes/robot_arms/fr3/visual/l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
- added link fr3_link3, mass 2.2449013699; collision mesh filename=package://franka_description/meshes/robot_arms/fr3/collisio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; visual mesh filename=package://franka_description/meshes/robot_arms/fr3/visual/l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
- added link fr3_link4, mass 2.6155955791; collision mesh filename=package://franka_description/meshes/robot_arms/fr3/collisio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; visual mesh filename=package://franka_description/meshes/robot_arms/fr3/visual/l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
- added link fr3_link5, mass 2.3271207594; collision mesh filename=package://franka_description/meshes/robot_arms/fr3/collisio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; visual mesh filename=package://franka_description/meshes/robot_arms/fr3/visual/l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
- added link fr3_link6, mass 1.8170376524; collision mesh filename=package://franka_description/meshes/robot_arms/fr3/collisio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; visual mesh filename=package://franka_description/meshes/robot_arms/fr3/visual/l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
- added link fr3_link7, mass 0.6271432862; collision mesh filename=package://franka_description/meshes/robot_arms/fr3/collisio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; visual mesh filename=package://franka_description/meshes/robot_arms/fr3/visual/l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
- link fr3_hand_sc: mass 0.73 -> None
- link fr3_link0_sc: mass 2.3966 -> None
- link fr3_link1_sc: mass 2.9274653454 -> None
- link fr3_link2_sc: mass 2.9355370338 -> None
- link fr3_link3_sc: mass 2.2449013699 -> None
- link fr3_link4_sc: mass 2.6155955791 -> None
- link fr3_link5_sc: mass 2.3271207594 -> None
- link fr3_link6_sc: mass 1.8170376524 -> None
- link fr3_link7_sc: mass 0.6271432862 -> None
Joints:
- removed joint fr3_joint0_sc
- added joint fr3_base_joint: type fixed, parent base, child fr3_link0, origin xyz=0 0 0 rpy=0 0 0
- added joint fr3_hand_sc_joint: type fixed, parent fr3_hand, child fr3_hand_sc, origin rpy=0 0 0
- added joint fr3_link0_sc_joint: type fixed, parent fr3_link0, child fr3_link0_sc, origin rpy=0 0 0
- added joint fr3_link1_sc_joint: type fixed, parent fr3_link1, child fr3_link1_sc, origin rpy=0 0 0
- added joint fr3_link2_sc_joint: type fixed, parent fr3_link2, child fr3_link2_sc, origin rpy=0 0 0
- added joint fr3_link3_sc_joint: type fixed, parent fr3_link3, child fr3_link3_sc, origin rpy=0 0 0
- added joint fr3_link4_sc_joint: type fixed, parent fr3_link4, child fr3_link4_sc, origin rpy=0 0 0
- added joint fr3_link5_sc_joint: type fixed, parent fr3_link5, child fr3_link5_sc, origin rpy=0 0 0
- added joint fr3_link6_sc_joint: type fixed, parent fr3_link6, child fr3_link6_sc, origin rpy=0 0 0
- added joint fr3_link7_sc_joint: type fixed, parent fr3_link7, child fr3_link7_sc, origin rpy=0 0 0.7853981633974483
- joint fr3_hand_joint: child fr3_hand_sc -> fr3_hand
- joint fr3_joint1: child fr3_link1_sc -> fr3_link1; parent fr3_link0_sc -> fr3_link0
- joint fr3_joint2: child fr3_link2_sc -> fr3_link2; parent fr3_link1_sc -> fr3_link1
- joint fr3_joint3: child fr3_link3_sc -> fr3_link3; parent fr3_link2_sc -> fr3_link2
- joint fr3_joint4: child fr3_link4_sc -> fr3_link4; parent fr3_link3_sc -> fr3_link3
- joint fr3_joint5: child fr3_link5_sc -> fr3_link5; parent fr3_link4_sc -> fr3_link4
- joint fr3_joint6: child fr3_link6_sc -> fr3_link6; parent fr3_link5_sc -> fr3_link5
- joint fr3_joint7: child fr3_link7_sc -> fr3_link7; parent fr3_link6_sc -> fr3_link6
- joint fr3_joint8: parent fr3_link7_sc -> fr3_link7

Commit message: 13microseconds_version

File: data/fr3_capsule.urdf (robot description, URDF)
Before this commit: robot fr3, 20 links, 19 joints
Links:
- removed link fr3_hand
- removed link fr3_link0
- removed link fr3_link1
- removed link fr3_link2
- removed link fr3_link3
- removed link fr3_link4
- removed link fr3_link5
- removed link fr3_link6
- removed link fr3_link7
- link fr3_hand_sc: mass None -> 0.73
- link fr3_link0_sc: mass None -> 2.3966
- link fr3_link1_sc: mass None -> 2.9274653454
- link fr3_link2_sc: mass None -> 2.9355370338
- link fr3_link3_sc: mass None -> 2.2449013699
- link fr3_link4_sc: mass None -> 2.6155955791
- link fr3_link5_sc: mass None -> 2.3271207594
- link fr3_link6_sc: mass None -> 1.8170376524
- link fr3_link7_sc: mass None -> 0.6271432862
Joints:
- removed joint fr3_base_joint
- removed joint fr3_hand_sc_joint
- removed joint fr3_link0_sc_joint
- removed joint fr3_link1_sc_joint
- removed joint fr3_link2_sc_joint
- removed joint fr3_link3_sc_joint
- removed joint fr3_link4_sc_joint
- removed joint fr3_link5_sc_joint
- removed joint fr3_link6_sc_joint
- removed joint fr3_link7_sc_joint
- added joint fr3_joint0_sc: type fixed, parent base, child fr3_link0_sc, origin xyz=0 0 0 rpy=0 0 0
- joint fr3_hand_joint: child fr3_hand -> fr3_hand_sc
- joint fr3_joint1: child fr3_link1 -> fr3_link1_sc; parent fr3_link0 -> fr3_link0_sc
- joint fr3_joint2: child fr3_link2 -> fr3_link2_sc; parent fr3_link1 -> fr3_link1_sc
- joint fr3_joint3: child fr3_link3 -> fr3_link3_sc; parent fr3_link2 -> fr3_link2_sc
- joint fr3_joint4: child fr3_link4 -> fr3_link4_sc; parent fr3_link3 -> fr3_link3_sc
- joint fr3_joint5: child fr3_link5 -> fr3_link5_sc; parent fr3_link4 -> fr3_link4_sc
- joint fr3_joint6: child fr3_link6 -> fr3_link6_sc; parent fr3_link5 -> fr3_link5_sc
- joint fr3_joint7: child fr3_link7 -> fr3_link7_sc; parent fr3_link6 -> fr3_link6_sc
- joint fr3_joint8: parent fr3_link7 -> fr3_link7_sc
